File: cad_files/Evezor_blank.kicad_pcb (KiCad board)
At the start: 2 copper layers, 49 x 65 mm, 37 parts, among them J1 USB_C_Receptacle_USB2.0, J2 RJ11, J3 RJ11, J4 PH, J5 PH, J6 Conn_02x03_Odd_Even, SW1 SW_Push, U1 SY8401ABC, U2 AMS1117-3.3, U3 EDGE_STM32F405_CPU_V1

Commit message: clean up fab layer
Parts:
- removed H1: MountingHole, Evezor_extras:OLED_STANDOFF
- C1, C3: value .1uF -> .1uF 100V; footprint Capacitor_SMD:C_0603_1608Metric -> Capacitor_SMD:C_0805_2012Metric
- C9: value C_Small -> .1uF
- R1: value 15k -> 10k
- moved C3 0.15 mm to (127.1, 142.6)
- moved C1 0.05 mm to (122.5, 139.7)
Routing:
- net GND: track 17.6 -> 18.9 mm
